File: KiCad/ESP32-C3-MINI-1-N4.kicad_sch (KiCad schematic)
At the start: 20 parts, among them U1 ESP32-C3-MINI-1-N4

Commit message: Fix LED's PNs
Parts:
- D1: value Green -> Yellow; MPN SZYY0603YG -> XL-0201UYC
- D2: MPN NCD0603R1 -> APG0603SURC-TT
- JP1, JP2, TP1: now left out of the parts list

Commit message: Widen servo traces, add C to slikscreen, replace LEDs to 0402
Parts:
- D1: footprint LED_SMD:LED_0201_0603Metric_Pad0.64x0.40mm_HandSolder -> LED_SMD:LED_0402_1005Metric_Pad0.77x0.64mm_HandSolder; MPN XL-0201UYC -> NCD0402Y1
- D2: footprint LED_SMD:LED_0201_0603Metric_Pad0.64x0.40mm_HandSolder -> LED_SMD:LED_0402_1005Metric_Pad0.77x0.64mm_HandSolder; MPN APG0603SURC-TT -> XL-1005SURC
Changed lines of the file:
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@@
     (title "Hydrofoil Control")
     (date "2023-09-04")
-    (rev "v1.0")
+    (rev "v1.1")
     (company "Tamás Nagy")
   )
