File: KiCad/Hydrofoil.kicad_sch (KiCad schematic)
At the start: 10 parts, among them J1 Conn_01x03_Pin, J2 Conn_01x03_Pin, U2 LD1117S33CTR, U3 TPS22917DBV

Commit message: Fix LED's PNs
Parts:
- J1, J2: now left out of the parts list

Commit message: Widen servo traces, add C to slikscreen, replace LEDs to 0402
Parts:
- added C10, C9: 10u, Capacitor_SMD:C_0402_1005Metric_Pad0.74x0.62mm_HandSolder, symbol Device:C
Connections:
- net +3.3V: now also C10.1
- net +5V: now also C9.1
- net GND: now also C10.2, C9.2
Other:
- moved on the sheet: C6
Changed lines of the file:
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@@
     (title "Hydrofoil Control")
     (date "2023-09-04")
-    (rev "v1.0")
+    (rev "v1.1")
     (company "Tamás Nagy")
   )
