File: KiCad/ADS1115-ADC.kicad_sch (KiCad schematic)
At the start: 32 parts, among them Q1 BSS138, Q2 BSS138, Q3 BSS138, Q4 BSS138, Q5 BSS138, U1 LM334M, U2 LM334M, U3 ADS1115IDGS

Commit message: Fix LED's PNs
Parts:
- CP1, CP2, CP3, CP4: now left out of the parts list
Changed lines of the file:
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@@
   )
   (symbol (lib_id "Connector:TestPoint") (at 96.52 166.37 180) (unit 1)
-    (in_bom yes) (on_board yes) (dnp no) (fields_autoplaced)
+    (in_bom no) (on_board yes) (dnp no) (fields_autoplaced)
     (property "Reference" "CP1" (at 99.06 168.402 0)
       (effects (font (size 1.27 1.27)) (justify right))
@@
   )
   (symbol (lib_id "Connector:TestPoint") (at 96.52 179.07 0) (unit 1)
-    (in_bom yes) (on_board yes) (dnp no) (fields_autoplaced)
+    (in_bom no) (on_board yes) (dnp no) (fields_autoplaced)
     (property "Reference" "CP2" (at 99.06 174.498 0)
       (effects (font (size 1.27 1.27)) (justify left))
@@
   )
   (symbol (lib_id "Connector:TestPoint") (at 138.43 179.07 0) (unit 1)
-    (in_bom yes) (on_board yes) (dnp no) (fields_autoplaced)
+    (in_bom no) (on_board yes) (dnp no) (fields_autoplaced)
     (property "Reference" "CP4" (at 140.97 174.498 0)
       (effects (font (size 1.27 1.27)) (justify left))
@@
   )
   (symbol (lib_id "Connector:TestPoint") (at 138.43 166.37 180) (unit 1)
-    (in_bom yes) (on_board yes) (dnp no) (fields_autoplaced)
+    (in_bom no) (on_board yes) (dnp no) (fields_autoplaced)
     (property "Reference" "CP3" (at 140.97 168.402 0)
       (effects (font (size 1.27 1.27)) (justify right))

Commit message: Add missing silkscreen texts
Parts:
- Q1, Q2, Q3, Q4, Q5: MPN BSS138 -> BSS138LT1G
Changed lines of the file:
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@@
       (effects (font (size 1.27 1.27)) (justify left) hide)
     )
-    (property "MPN" "BSS138" (at 162.56 58.42 90)
+    (property "MPN" "BSS138LT1G" (at 162.56 58.42 90)
       (effects (font (size 1.27 1.27)) hide)
     )
@@
       (effects (font (size 1.27 1.27)) (justify left) hide)
     )
-    (property "MPN" "BSS138" (at 240.03 93.98 90)
+    (property "MPN" "BSS138LT1G" (at 240.03 93.98 90)
       (effects (font (size 1.27 1.27)) hide)
     )
@@
       (effects (font (size 1.27 1.27)) (justify left) hide)
     )
-    (property "MPN" "BSS138" (at 240.03 58.42 90)
+    (property "MPN" "BSS138LT1G" (at 240.03 58.42 90)
       (effects (font (size 1.27 1.27)) hide)
     )
@@
       (effects (font (size 1.27 1.27)) (justify left) hide)
     )
-    (property "MPN" "BSS138" (at 162.56 93.98 90)
+    (property "MPN" "BSS138LT1G" (at 162.56 93.98 90)
       (effects (font (size 1.27 1.27)) hide)
     )
@@
       (effects (font (size 1.27 1.27)) (justify left) hide)
     )
-    (property "MPN" "BSS138" (at 240.03 133.35 90)
-      (effects (font (size 1.27 1.27)) hide)
-    )
+    (property "MPN" "BSS138LT1G" (at 240.03 133.35 90)
+      (effects (font (size 1.27 1.27)) hide)
+    )
